Commit message: fix the problem that roll disappear, but mid360 still fails to load in rviz

File: src/wheeltec_robot_gazebo/wheeltec_description/urdf/mini_mec/minimec_rplidar.xacro (robot description, xacro)
@@ -48,5 +48,5 @@
                 </ray>
                 <plugin name="gazebo_rplidar" filename="libgazebo_ros_laser.so">
-                    <topicName>/scan</topicName>
+                    <topicName>scan</topicName>
                     <frameName>laser_link</frameName>
                 </plugin>

File: src/wheeltec_robot_gazebo/wheeltec_description/urdf/mini_mec/my_mini_mec.xacro (robot description, xacro)
@@ -8,5 +8,6 @@
     <xacro:property name="rplidar_offset_x" value="0.048632" />
     <xacro:property name="rplidar_offset_y" value="0.00018237" />
-    <xacro:property name="rplidar_offset_z" value="0.1296" />
+    <!-- <xacro:property name="rplidar_offset_z" value="0.1296" /> -->
+    <xacro:property name="rplidar_offset_z" value="0.0796" />
     <!--rplidar scanning angle-->
     <xacro:property name="rplidar_min_angle" value="-180" />
@@ -40,12 +41,15 @@
     <!-- <xacro:include filename="$(find wheeltec_description)/urdf/mini_mec/minimec_rplidar.xacro" /> -->
     <!-- <xacro:include filename="$(find wheeltec_description)/urdf/mini_mec/minimec_camera.xacro" /> -->
+    <xacro:include filename="$(find wheeltec_description)/urdf/livox_mid360.xacro" />
     <xacro:include filename="$(find wheeltec_description)/urdf/imu.xacro" />
     <xacro:include filename="$(find wheeltec_description)/urdf/material.xacro" />
     <xacro:include filename="$(find wheeltec_description)/urdf/mini_mec/my_minimec_transmission.xacro" />
-    <!-- <joint name="rplidar_joint" type="fixed">
-        <origin xyz="${rplidar_offset_x} ${rplidar_offset_y} ${rplidar_offset_z}" rpy="0 0 0" />
+    <xacro:laser_livox LA="laser"/>
+    <!-- <xacro:Livox_Mid360 name="laser_link"/> -->
+    <joint name="laser_joint" type="fixed">
+        <origin xyz="${rplidar_offset_x} ${rplidar_offset_y} ${rplidar_offset_z}" rpy="0 0 ${M_PI}" />
         <parent link="base_link"/>
         <child link="laser_link"/>
-    </joint> -->
+    </joint>
     <!-- Attach the camera -->
     <!-- <joint name="camera_frame_joint" type="fixed">

File: src/wheeltec_robot_gazebo/wheeltec_description/urdf/mini_mec/my_minimec_transmission.xacro (robot description, xacro)
@@ -26,8 +26,8 @@
       <type>transmission_interface/SimpleTransmission</type>
       <joint name="${LR}_${FR}_wheel_joint">
-        <hardwareInterface>VelocityJointInterface</hardwareInterface>
+        <hardwareInterface>hardware_interface/VelocityJointInterface</hardwareInterface>
       </joint>
       <actuator name="${LR}_${FR}_wheel_joint_motor">
-        <hardwareInterface>VelocityJointInterface</hardwareInterface>
+        <hardwareInterface>hardware_interface/VelocityJointInterface</hardwareInterface>
         <mechanicalReduction>1</mechanicalReduction>
         <motorTorqueConstant>1</motorTorqueConstant>

File: src/wheeltec_robot_gazebo/wheeltec_description/urdf/mini_mec_control/minimec_transmission.xacro (robot description, xacro)
@@ -42,7 +42,7 @@
       <max_turn>3</max_turn>
       <!--ROS: Subscribe to the velocity command topic (usually "cmd_vel")-->
-      <commandTopic>/cmd_vel</commandTopic>
+      <commandTopic>cmd_vel</commandTopic>
       <!--ROS: Publish to the odometry topic (usually "odom")-->
-      <odometryTopic>/odom</odometryTopic>
+      <odometryTopic>odom</odometryTopic>
       <!--tf connect odometryFrame to robotBaseFrame-->
       <odometryFrame>odom</odometryFrame>
