Commit message: fixed mid360 bug, however one ugv can use for the fixed topic

File: src/wheeltec_robot_gazebo/wheeltec_description/urdf/livox_mid360.xacro (robot description, xacro)
@@ -2,19 +2,30 @@
 <robot name="wheeltec"
     xmlns:xacro="http://www.ros.org/wiki/xacro">
+    <xacro:property name="update_rate" value="20"/>
+    <xacro:property name="resolution" value="0.01"/>
+    <xacro:property name="noise_mean" value="0.01"/>
+    <xacro:property name="noise_stddev" value="0.00"/>
+    <xacro:property name="laser_min_range" value="0.1"/>
+    <xacro:property name="laser_max_range" value="200"/>
+    <xacro:property name="samples" value="20000"/>
+    <xacro:property name="downsample" value="1"/>
     <xacro:macro name="laser_livox" params="LA">
         <link name="laser_link">
+            <inertial>
+                <mass value="0.114"/>
+                <origin xyz="0 0 0"/>
+                <inertia ixx="0.001" ixy="0.0" ixz="0.0" iyy="0.001" iyz="0.0" izz="0.001"/>
+            </inertial>
             <visual>
                 <origin xyz="0 0 0" rpy="0 0 0"/>
                 <geometry>
-                    <!-- <box size="0.05 0.05 0.05"/> -->
-                    <mesh filename="package://wheeltec_description/meshes/livox_mid360/livox_mid-360-90x.dae" />
+                    <mesh filename="package://wheeltec_description/meshes/livox_mid360/livox_mid360.stl" scale="1 1 1"/>
                 </geometry>
-                <material name="black"/>
             </visual>
             <collision>
-                <origin xyz="0 0 0" rpy="0 0 0"/>
                 <geometry>
-                    <!-- <box size="0.05 0.05 0.05"/> -->
-                    <mesh filename="package://wheeltec_description/meshes/livox_mid360/livox_mid-360-90x.dae" />
+                    <box>
+                        <size>0.05 0.05 0.05</size>
+                    </box>
                 </geometry>
             </collision>
@@ -25,7 +36,7 @@
             <!--define sensor-->
             <sensor type="ray" name="laser_livox">
-                <visualize>True</visualize>
+                <visualize>false</visualize>
                 <always_on>True</always_on>
-                <update_rate>20</update_rate>
+                <update_rate>${update_rate}</update_rate>
                 <plugin name="gazebo_ros_laser_controller" filename="liblivox_laser_simulation.so">
                     <ray>
@@ -34,29 +45,29 @@
                                 <samples>100</samples>
                                 <resolution>1</resolution>
-                                <min_angle>-3.1415926535897931</min_angle>
-                                <max_angle>3.1415926535897931</max_angle>
+                                <min_angle>-${M_PI}</min_angle>
+                                <max_angle>${M_PI}</max_angle>
                             </horizontal>
                             <vertical>
-                                <samples>50</samples>
+                                <samples>100</samples>
                                 <resolution>1</resolution>
-                                <min_angle>-3.1415926535897931</min_angle>
-                                <max_angle>3.1415926535897931</max_angle>
+                                <min_angle>${-7.22/180*M_PI}</min_angle>
+                                <max_angle>${55.22/180*M_PI}</max_angle>
                             </vertical>
                         </scan>
                         <range>
-                            <min>0.1</min>
-                            <max>40</max>
-                            <resolution>1</resolution>
+                            <min>${laser_min_range}</min>
+                            <max>${laser_max_range}</max>
+                            <resolution>${resolution}</resolution>
                         </range>
                         <noise>
                             <type>gaussian</type>
-                            <mean>0.0</mean>
-                            <stddev>0.0</stddev>
+                            <mean>${noise_mean}</mean>
+                            <stddev>${resolution}</stddev>
                         </noise>
                     </ray>
                     <visualize>True</visualize>
-                    <samples>20000</samples>
-                    <downsample>1</downsample>
-                    <csv_file_name>mid360-real-centr.csv</csv_file_name>
+                    <samples>${samples}</samples>
+                    <downsample>${downsample}</downsample>
+                    <csv_file_name>package://wheeltec_description/meshes/livox_mid360/mid360.csv</csv_file_name>
                     <publish_pointcloud_type>2</publish_pointcloud_type>
                     <ros_topic>ugv_1/lidar</ros_topic>

File: src/wheeltec_robot_gazebo/wheeltec_description/urdf/mini_mec/my_mini_mec.xacro (robot description, xacro)
@@ -8,6 +8,5 @@
     <xacro:property name="rplidar_offset_x" value="0.048632" />
     <xacro:property name="rplidar_offset_y" value="0.00018237" />
-    <!-- <xacro:property name="rplidar_offset_z" value="0.1296" /> -->
-    <xacro:property name="rplidar_offset_z" value="0.0796" />
+    <xacro:property name="rplidar_offset_z" value="0.0996" />
     <!--rplidar scanning angle-->
     <xacro:property name="rplidar_min_angle" value="-180" />
@@ -46,7 +45,6 @@
     <xacro:include filename="$(find wheeltec_description)/urdf/mini_mec/my_minimec_transmission.xacro" />
     <xacro:laser_livox LA="laser"/>
-    <!-- <xacro:Livox_Mid360 name="laser_link"/> -->
     <joint name="laser_joint" type="fixed">
-        <origin xyz="${rplidar_offset_x} ${rplidar_offset_y} ${rplidar_offset_z}" rpy="0 0 ${M_PI}" />
+        <origin xyz="${rplidar_offset_x} ${rplidar_offset_y} ${rplidar_offset_z}" rpy="0 0 0" />
         <parent link="base_link"/>
         <child link="laser_link"/>

Commit message: the topic and frameid of mid360 can change dynamicly according to the ns of UGV

File: src/wheeltec_robot_gazebo/wheeltec_description/urdf/livox_mid360.xacro (robot description, xacro)
@@ -10,5 +10,5 @@
     <xacro:property name="samples" value="20000"/>
     <xacro:property name="downsample" value="1"/>
-    <xacro:macro name="laser_livox" params="LA">
+    <xacro:macro name="laser_livox" params="NS">
         <link name="laser_link">
             <inertial>
@@ -71,6 +71,6 @@
                     <csv_file_name>package://wheeltec_description/meshes/livox_mid360/mid360.csv</csv_file_name>
                     <publish_pointcloud_type>2</publish_pointcloud_type>
-                    <ros_topic>ugv_1/lidar</ros_topic>
-                    <frameName>ugv_1/laser_link</frameName>
+                    <ros_topic>${NS}/lidar</ros_topic>
+                    <frameName>${NS}/laser_link</frameName>
                 </plugin>
             </sensor>

File: src/wheeltec_robot_gazebo/wheeltec_description/urdf/mini_mec/my_mini_mec.xacro (robot description, xacro)
@@ -2,4 +2,5 @@
 <robot name="wheeltec"
     xmlns:xacro="http://www.ros.org/wiki/xacro">
+    <xacro:property name="namespace" value="$(arg namespace)"/>
     <!--M_PI-->
     <xacro:property name="M_PI" value="3.1415926535897931" />
@@ -44,5 +45,5 @@
     <xacro:include filename="$(find wheeltec_description)/urdf/material.xacro" />
     <xacro:include filename="$(find wheeltec_description)/urdf/mini_mec/my_minimec_transmission.xacro" />
-    <xacro:laser_livox LA="laser"/>
+    <xacro:laser_livox NS="${namespace}"/>
     <joint name="laser_joint" type="fixed">
         <origin xyz="${rplidar_offset_x} ${rplidar_offset_y} ${rplidar_offset_z}" rpy="0 0 0" />

Commit message: fix the problem of lidar angle

File: src/wheeltec_robot_gazebo/wheeltec_description/urdf/livox_mid360.xacro (robot description, xacro)
@@ -7,5 +7,5 @@
     <xacro:property name="noise_stddev" value="0.00"/>
     <xacro:property name="laser_min_range" value="0.1"/>
-    <xacro:property name="laser_max_range" value="200"/>
+    <xacro:property name="laser_max_range" value="40"/>
     <xacro:property name="samples" value="20000"/>
     <xacro:property name="downsample" value="1"/>
@@ -24,4 +24,5 @@
             </visual>
             <collision>
+                <origin xyz="0 0 0" rpy="0 0 0"/>
                 <geometry>
                     <box>
@@ -36,5 +37,5 @@
             <!--define sensor-->
             <sensor type="ray" name="laser_livox">
-                <visualize>false</visualize>
+                <visualize>true</visualize>
                 <always_on>True</always_on>
                 <update_rate>${update_rate}</update_rate>
@@ -51,6 +52,6 @@
                                 <samples>100</samples>
                                 <resolution>1</resolution>
-                                <min_angle>${-7.22/180*M_PI}</min_angle>
-                                <max_angle>${55.22/180*M_PI}</max_angle>
+                                <min_angle>${-M_PI}</min_angle>
+                                <max_angle>${M_PI}</max_angle>
                             </vertical>
                         </scan>

Commit message: 4 robots simu version, use gazebo/link_states base_footprin's ofom and mid360-generated sensor_msgs::pointcloud2, which can replace the MR_SLAM(FAST-LIO) in real world

File: src/wheeltec_robot_gazebo/wheeltec_description/urdf/livox_mid360.xacro (robot description, xacro)
@@ -2,5 +2,5 @@
 <robot name="wheeltec"
     xmlns:xacro="http://www.ros.org/wiki/xacro">
-    <xacro:property name="update_rate" value="20"/>
+    <xacro:property name="update_rate" value="30"/>
     <xacro:property name="resolution" value="0.01"/>
     <xacro:property name="noise_mean" value="0.01"/>
@@ -37,5 +37,5 @@
             <!--define sensor-->
             <sensor type="ray" name="laser_livox">
-                <visualize>true</visualize>
+                <visualize>false</visualize>
                 <always_on>True</always_on>
                 <update_rate>${update_rate}</update_rate>

Commit message: update

File: src/wheeltec_robot_gazebo/wheeltec_description/urdf/livox_mid360.xacro (robot description, xacro)
@@ -8,5 +8,5 @@
     <xacro:property name="laser_min_range" value="0.1"/>
     <xacro:property name="laser_max_range" value="40"/>
-    <xacro:property name="samples" value="20000"/>
+    <xacro:property name="samples" value="6000"/>
     <xacro:property name="downsample" value="1"/>
     <xacro:macro name="laser_livox" params="NS">
@@ -44,5 +44,5 @@
                         <scan>
                             <horizontal>
-                                <samples>100</samples>
+                                <samples>50</samples>
                                 <resolution>1</resolution>
                                 <min_angle>-${M_PI}</min_angle>
@@ -50,5 +50,5 @@
                             </horizontal>
                             <vertical>
-                                <samples>100</samples>
+                                <samples>50</samples>
                                 <resolution>1</resolution>
                                 <min_angle>${-M_PI}</min_angle>

File: src/wheeltec_robot_gazebo/wheeltec_description/urdf/mini_mec/my_mini_mec.xacro (robot description, xacro)
@@ -27,6 +27,6 @@
     <xacro:property name="wheel_position_z" value="-0.036" />
     <xacro:property name="rear_wheel_position_x" value="-0.087868" />
-    <xacro:property name="wheel_mass" value="0.026412" />
-    <xacro:property name="shaft_mass" value="0.00016066" />
+    <xacro:property name="wheel_mass" value="1.622412" />
+    <xacro:property name="shaft_mass" value="0.0016066" />
     <xacro:property name="roll_mass" value="0.0023973" />
     <xacro:property name="box_position_x" value="0" />
@@ -36,5 +36,5 @@
     <xacro:property name="box_height" value="0.07" />
     <xacro:property name="box_width" value="0.12" />
-    <xacro:property name="box_mass" value="0.082" />
+    <xacro:property name="box_mass" value="1.982" />
     <!--robot with rplidar and camera -->
     <xacro:include filename="$(find wheeltec_description)/urdf/mini_mec/minimec_body.xacro" />
@@ -63,5 +63,5 @@
             <child link="${LR}_${FR}_wheel_link"/>
             <axis xyz="0 1 0" rpy="0 0 0"/>
-            <limit effort="3.9" velocity="36.92"/>
+            <limit effort="15" velocity="56.92"/>
         </joint>
     </xacro:macro>
